Commit message: feat: ros2_control hw

File: gerbil_description/urdf/mobile_base.ros2_control.xacro (robot description, xacro)
@@ -6,10 +6,10 @@
             <param name="calculate_dyamics" value="true"/>
         </hardware>
-        <joint name="base_right_wheel_joint">
+        <joint name="base_left_wheel_joint">
             <command_interface name="velocity"/>
             <state_interface name="velocity"/>
             <state_interface name="position"/>
         </joint>
-        <joint name="base_left_wheel_joint">
+        <joint name="base_right_wheel_joint">
             <command_interface name="velocity"/>
             <state_interface name="velocity"/>

Commit message: changes to urdf to include intertia and collision values, changes to ensure TODOs on wheel seperations for actual measurment for wheels, imu xyz position, and add comments/mock hardware if/else

File: gerbil_description/urdf/mobile_base.ros2_control.xacro (robot description, xacro)
@@ -1,17 +1,26 @@
 <?xml version="1.0"?>
 <robot xmlns:xacro="http://www.ros.org/wiki/xacro">
+    <!-- Hardware mode: 'mock' for simulation, 'real' for actual RoboClaw -->
+    <xacro:arg name="use_mock_hardware" default="true" />
     <ros2_control name="GerbilRoboClawSystem" type="system">
-        <!-- this is mock hardware for simulation or testing without actual roboclaw hardware -->
-        <hardware>
-            <plugin>mock_components/GenericSystem</plugin>
-        </hardware>
-        <!-- this is the actual roboclaw hardware, comment this out if your not sshed into jetson -->
-        <!-- <hardware>
-            <plugin>gerbil_hw/RoboClawHardwareInterface</plugin>
-            <param name="serial_port">/dev/roboclaw</param>
-        </hardware> -->
+        <!-- Mock hardware for simulation or testing without actual RoboClaw -->
+        <xacro:if value="$(arg use_mock_hardware)">
+            <hardware>
+                <plugin>mock_components/GenericSystem</plugin>
+            </hardware>
+        </xacro:if>
+        <!-- Real RoboClaw hardware (use when SSH'd into Jetson) -->
+        <xacro:unless value="$(arg use_mock_hardware)">
+            <hardware>
+                <plugin>gerbil_hw/RoboClawHardwareInterface</plugin>
+                <param name="serial_port">/dev/ttyTHS1</param>
+            </hardware>
+        </xacro:unless>
         <!-- joints that are defined and do not change whether using mock hardware or actual roboclaw hardware -->
         <joint name="base_left_wheel_joint">
-            <command_interface name="velocity"/>
+            <command_interface name="velocity">
+                <param name="min">-10.0</param>
+                <param name="max">10.0</param>
+            </command_interface>
             <state_interface name="position"/>
             <state_interface name="velocity"/>
@@ -22,5 +31,8 @@
         </joint>
         <joint name="base_right_wheel_joint">
-            <command_interface name="velocity"/>
+            <command_interface name="velocity">
+                <param name="min">-10.0</param>
+                <param name="max">10.0</param>
+            </command_interface>
             <state_interface name="position"/>
             <state_interface name="velocity"/>

File: gerbil_description/urdf/mobile_base.xacro (robot description, xacro)
@@ -1,10 +1,18 @@
 <?xml version="1.0"?>
 <robot xmlns:xacro="http://www.ros.org/wiki/xacro">
-    <xacro:property name="base_length" value="0.6" />
-    <xacro:property name="base_width" value="0.4" />
-    <xacro:property name="base_height" value="0.2" />
-    <xacro:property name="wheel_radius" value="0.1" />
-    <xacro:property name="wheel_length" value="0.05" />
+    <!-- ==================== ROBOT DIMENSIONS ==================== -->
+    <!-- TODO: Update these values with actual measurements from your robot -->
+    <xacro:property name="base_length" value="0.6" />      <!-- meters (front to back) -->
+    <xacro:property name="base_width" value="0.4" />       <!-- meters (side to side, excluding wheels) -->
+    <xacro:property name="base_height" value="0.2" />      <!-- meters -->
+    <xacro:property name="base_mass" value="5.0" />        <!-- kg -->
+    <xacro:property name="wheel_radius" value="0.1" />     <!-- meters -->
+    <xacro:property name="wheel_length" value="0.05" />    <!-- meters (wheel width) -->
+    <xacro:property name="wheel_mass" value="0.5" />       <!-- kg -->
+    <!-- Calculated wheel separation (center to center) -->
+    <xacro:property name="wheel_separation" value="${base_width + wheel_length}" />
+    <!-- ==================== BASE FOOTPRINT ==================== -->
     <link name="base_footprint" />
+    <!-- ==================== BASE LINK ==================== -->
     <link name="base_link">
         <visual>
@@ -15,5 +23,21 @@
             <material name="blue" />
         </visual>
+        <collision>
+            <geometry>
+                <box size="${base_length} ${base_width} ${base_height}" />
+            </geometry>
+            <origin xyz="0 0 ${base_height / 2.0}" rpy="0 0 0" />
+        </collision>
+        <inertial>
+            <mass value="${base_mass}" />
+            <origin xyz="0 0 ${base_height / 2.0}" rpy="0 0 0" />
+            <inertia ixx="${(1/12) * base_mass * (base_width*base_width + base_height*base_height)}"
+                     ixy="0" ixz="0"
+                     iyy="${(1/12) * base_mass * (base_length*base_length + base_height*base_height)}"
+                     iyz="0"
+                     izz="${(1/12) * base_mass * (base_length*base_length + base_width*base_width)}" />
+        </inertial>
     </link>
+    <!-- ==================== WHEEL MACRO ==================== -->
     <xacro:macro name="wheel_link" params="prefix">
         <link name="${prefix}_wheel_link">
@@ -25,8 +49,24 @@
                 <material name="grey" />
             </visual>
+            <collision>
+                <geometry>
+                    <cylinder radius="${wheel_radius}" length="${wheel_length}" />
+                </geometry>
+                <origin xyz="0 0 0" rpy="${pi / 2.0} 0 0" />
+            </collision>
+            <inertial>
+                <mass value="${wheel_mass}" />
+                <origin xyz="0 0 0" rpy="${pi / 2.0} 0 0" />
+                <inertia ixx="${(1/12) * wheel_mass * (3*wheel_radius*wheel_radius + wheel_length*wheel_length)}"
+                         ixy="0" ixz="0"
+                         iyy="${(1/12) * wheel_mass * (3*wheel_radius*wheel_radius + wheel_length*wheel_length)}"
+                         iyz="0"
+                         izz="${(1/2) * wheel_mass * wheel_radius*wheel_radius}" />
+            </inertial>
         </link>
     </xacro:macro>
     <xacro:wheel_link prefix="right" />
     <xacro:wheel_link prefix="left" />
+    <!-- ==================== CASTER WHEEL ==================== -->
     <link name="caster_wheel_link">
         <visual>
@@ -37,5 +77,38 @@
             <material name="grey" />
         </visual>
+        <collision>
+            <geometry>
+                <sphere radius="${wheel_radius / 2.0}" />
+            </geometry>
+            <origin xyz="0 0 0" rpy="0 0 0" />
+        </collision>
+        <inertial>
+            <mass value="0.2" />
+            <origin xyz="0 0 0" rpy="0 0 0" />
+            <inertia ixx="0.0001" ixy="0" ixz="0" iyy="0.0001" iyz="0" izz="0.0001" />
+        </inertial>
     </link>
+    <!-- ==================== IMU LINK ==================== -->
+    <link name="imu_link">
+        <visual>
+            <geometry>
+                <box size="0.03 0.03 0.01" />
+            </geometry>
+            <origin xyz="0 0 0" rpy="0 0 0" />
+            <material name="green">
+                <color rgba="0 1 0 1" />
+            </material>
+        </visual>
+        <collision>
+            <geometry>
+                <box size="0.03 0.03 0.01" />
+            </geometry>
+        </collision>
+        <inertial>
+            <mass value="0.01" />
+            <inertia ixx="0.000001" ixy="0" ixz="0" iyy="0.000001" iyz="0" izz="0.000001" />
+        </inertial>
+    </link>
+    <!-- ==================== JOINTS ==================== -->
     <joint name="base_joint" type="fixed">
         <parent link="base_footprint" />
@@ -60,3 +133,10 @@
         <origin xyz="${base_length / 3.0} 0 ${-wheel_radius / 2.0}" rpy="0 0 0" />
     </joint>
+    <!-- IMU mounted on top of base_link -->
+    <!-- TODO: Adjust xyz to match actual IMU position on your robot -->
+    <joint name="imu_joint" type="fixed">
+        <parent link="base_link" />
+        <child link="imu_link" />
+        <origin xyz="0 0 ${base_height}" rpy="0 0 0" />
+    </joint>
 </robot>
