Commit message: made changes to allow for duty cycle control of motors, no encoders are used, but PID can be enabled when configured in Motion Studio, for now this is okay, I believe encoders might not even be that useful but anything helps

File: src/gerbil_description/urdf/mobile_base.ros2_control.xacro (robot description, xacro)
@@ -1,5 +1,5 @@
 <?xml version="1.0"?>
 <robot xmlns:xacro="http://www.ros.org/wiki/xacro">
-    <!-- Hardware mode: 'mock' for simulation, 'real' for actual RoboClaw -->
+    <!-- Hardware mode - mock for simulation, real for actual RoboClaw -->
     <xacro:arg name="use_mock_hardware" default="true" />
     <ros2_control name="GerbilRoboClawSystem" type="system">
@@ -15,4 +15,7 @@
                 <plugin>gerbil_hw/RoboClawHardwareInterface</plugin>
                 <param name="serial_port">/dev/ttyTHS1</param>
+                <!-- Duty cycle mode - bypasses velocity PID, no encoders needed -->
+                <!-- Set to false once encoders are wired up -->
+                <param name="use_duty_cycle">true</param>
             </hardware>
         </xacro:unless>
@@ -24,8 +27,9 @@
             </command_interface>
             <state_interface name="position"/>
-            <!-- TODO Verify these parameters -->
             <param name="address">128</param>
             <param name="qppr">500</param>
             <param name="motor_type">M2</param>
+            <!-- Motor speed (rad/s) that maps to 100 percent duty cycle. Lower = more responsive -->
+            <param name="max_duty_speed">10.0</param>
         </joint>
         <joint name="base_right_wheel_joint">
@@ -35,8 +39,9 @@
             </command_interface>
             <state_interface name="position"/>
-            <!-- TODO Verify these parameters -->
             <param name="address">128</param>
             <param name="qppr">500</param>
             <param name="motor_type">M1</param>
+            <!-- Motor speed (rad/s) that maps to 100 percent duty cycle. Lower = more responsive -->
+            <param name="max_duty_speed">10.0</param>
         </joint>
     </ros2_control>

File: src/gerbil_description/urdf/mobile_base.xacro (robot description, xacro)
@@ -1,18 +1,20 @@
 <?xml version="1.0"?>
 <robot xmlns:xacro="http://www.ros.org/wiki/xacro">
-    <!-- ==================== ROBOT DIMENSIONS ==================== -->
-    <!-- TODO Update these values with actual measurements from your robot -->
-    <xacro:property name="base_length" value="0.6" />      <!-- meters (front to back) -->
-    <xacro:property name="base_width" value="0.4" />       <!-- meters (side to side, excluding wheels) -->
-    <xacro:property name="base_height" value="0.2" />      <!-- meters -->
-    <xacro:property name="base_mass" value="5.0" />        <!-- kg -->
-    <xacro:property name="wheel_radius" value="0.1" />     <!-- meters -->
-    <xacro:property name="wheel_length" value="0.05" />    <!-- meters (wheel width) -->
-    <xacro:property name="wheel_mass" value="0.5" />       <!-- kg -->
-    <!-- Calculated wheel separation (center to center) -->
-    <xacro:property name="wheel_separation" value="${base_width + wheel_length}" />
-    <!-- ==================== BASE FOOTPRINT ==================== -->
+    <!-- ROBOT DIMENSIONS -->
+    <!-- Drive wheels and ZED camera are at the front (+X) -->
+    <!-- Caster wheel is at the rear (-X) -->
+    <xacro:property name="base_length" value="0.6096" />      <!-- 24 inches -->
+    <xacro:property name="base_width" value="0.3048" />       <!-- 12 inches -->
+    <xacro:property name="base_height" value="0.0635" />      <!-- 2.5 inches -->
+    <xacro:property name="base_mass" value="6.8" />           <!-- ~15 lbs -->
+    <xacro:property name="wheel_radius" value="0.04756" />    <!-- 95.11mm diameter -->
+    <xacro:property name="wheel_length" value="0.03195" />    <!-- 31.95mm width -->
+    <xacro:property name="wheel_mass" value="0.5" />          <!-- kg estimate -->
+    <xacro:property name="wheel_separation" value="0.42285" /> <!-- 422.85mm center-to-center -->
+    <!-- Wheel X position - near front edge of chassis -->
+    <xacro:property name="wheel_x_offset" value="${base_length / 2.0 - 0.06}" />
+    <!-- BASE FOOTPRINT -->
     <link name="base_footprint" />
-    <!-- ==================== BASE LINK ==================== -->
+    <!-- BASE LINK -->
     <link name="base_link">
         <visual>
@@ -39,5 +41,5 @@
         </inertial>
     </link>
-    <!-- ==================== WHEEL MACRO ==================== -->
+    <!-- WHEEL MACRO -->
     <xacro:macro name="wheel_link" params="prefix">
         <link name="${prefix}_wheel_link">
@@ -68,5 +70,5 @@
     <xacro:wheel_link prefix="right" />
     <xacro:wheel_link prefix="left" />
-    <!-- ==================== CASTER WHEEL ==================== -->
+    <!-- CASTER WHEEL -->
     <link name="caster_wheel_link">
         <visual>
@@ -89,5 +91,5 @@
         </inertial>
     </link>
-    <!-- ==================== IMU LINK ==================== -->
+    <!-- IMU LINK -->
     <link name="imu_link">
         <visual>
@@ -110,5 +112,28 @@
         </inertial>
     </link>
-    <!-- ==================== JOINTS ==================== -->
+    <!-- ZED2i CAMERA LINK -->
+    <!-- Named 'zed_camera_link' to match the ZED wrapper's TF frame,
+         connecting the robot URDF tree to the ZED's internal frame chain -->
+    <link name="zed_camera_link">
+        <visual>
+            <geometry>
+                <box size="0.033 0.175 0.030" />
+            </geometry>
+            <origin xyz="0 0 0" rpy="0 0 0" />
+            <material name="dark_grey">
+                <color rgba="0.2 0.2 0.2 1" />
+            </material>
+        </visual>
+        <collision>
+            <geometry>
+                <box size="0.033 0.175 0.030" />
+            </geometry>
+        </collision>
+        <inertial>
+            <mass value="0.175" />
+            <inertia ixx="0.000001" ixy="0" ixz="0" iyy="0.000001" iyz="0" izz="0.000001" />
+        </inertial>
+    </link>
+    <!-- JOINTS -->
     <joint name="base_joint" type="fixed">
         <parent link="base_footprint" />
@@ -116,8 +141,9 @@
         <origin xyz="0 0 ${wheel_radius}" rpy="0 0 0"/>
     </joint>
+    <!-- Drive wheels at rear but changed to front -->
     <joint name="base_right_wheel_joint" type="continuous">
         <parent link="base_link" />
         <child link="right_wheel_link" />
-        <origin xyz="${-base_length / 4.0} ${-(base_width + wheel_length) / 2.0} 0" rpy="0 0 0" />
+        <origin xyz="${wheel_x_offset} ${-wheel_separation / 2.0} 0" rpy="0 0 0" />
         <axis xyz="0 1 0" />
     </joint>
@@ -125,18 +151,24 @@
         <parent link="base_link" />
         <child link="left_wheel_link" />
-        <origin xyz="${-base_length / 4.0} ${(base_width + wheel_length) / 2.0} 0" rpy="0 0 0" />
+        <origin xyz="${wheel_x_offset} ${wheel_separation / 2.0} 0" rpy="0 0 0" />
         <axis xyz="0 1 0" />
     </joint>
+    <!-- Caster at the front, but we consider it rear -->
     <joint name="base_caster_wheel_joint" type="fixed">
         <parent link="base_link" />
         <child link="caster_wheel_link" />
-        <origin xyz="${base_length / 3.0} 0 ${-wheel_radius / 2.0}" rpy="0 0 0" />
+        <origin xyz="${-wheel_x_offset} 0 ${-wheel_radius / 2.0}" rpy="0 0 0" />
     </joint>
-    <!-- IMU mounted on top of base_link -->
-    <!-- TODO Adjust xyz to match actual IMU position on your robot -->
+    <!-- IMU centered on top of chassis not quite right, doesn't really matter, can add meshes later -->
     <joint name="imu_joint" type="fixed">
         <parent link="base_link" />
         <child link="imu_link" />
-        <origin xyz="0 0 ${base_height}" rpy="0 0 0" />
+        <origin xyz="0 0 ${base_height + 0.005}" rpy="0 0 0" />
+    </joint>
+    <!-- ZED camera at front edge, on top of chassis, facing forward (rear) -->
+    <joint name="camera_joint" type="fixed">
+        <parent link="base_link" />
+        <child link="zed_camera_link" />
+        <origin xyz="${base_length / 2.0 - 0.02} 0 ${base_height + 0.015}" rpy="0 0 0" />
     </joint>
 </robot>
