Commit message: feat: migration to ZED SDK 5.2, total redownload in vendors directory

File: src/vendors/zed_wrapper/zed_wrapper/urdf/zed_macro.urdf.xacro (robot description, xacro)
@@ -1,5 +1,5 @@
 <?xml version="1.0"?>
 <!--
-// Copyright 2024 Stereolabs
+// Copyright 2025 Stereolabs
 //
 // Licensed under the Apache License, Version 2.0 (the "License");
@@ -16,5 +16,4 @@
 -->
 <robot xmlns:xacro="http://wiki.ros.org/xacro">
-  <xacro:include filename="$(find zed_wrapper)/urdf/include/materials.urdf.xacro" />
   <xacro:property name="M_PI"     value="3.1415926535897931" />
   <!--
@@ -33,4 +32,5 @@
       <xacro:property name="optical_offset_x" value="-0.01" />
       <xacro:property name="mono" value="false" />
+      <xacro:property name="mat" value="0.8 0.8 0.8 1.0" />
     </xacro:if>
     <xacro:if value="${model == 'zedm'}">
@@ -42,4 +42,5 @@
       <xacro:property name="optical_offset_x" value="0.0" />
       <xacro:property name="mono" value="false" />
+      <xacro:property name="mat" value="0 0 0 1.0" />
     </xacro:if>
     <xacro:if value="${model == 'zed2'}">
@@ -51,4 +52,5 @@
       <xacro:property name="optical_offset_x" value="-0.01" />
       <xacro:property name="mono" value="false" />
+      <xacro:property name="mat" value="0.25 0.25 0.25 1.0" />
     </xacro:if>
     <xacro:if value="${model == 'zed2i'}">
@@ -60,4 +62,5 @@
       <xacro:property name="optical_offset_x" value="-0.01" />
       <xacro:property name="mono" value="false" />
+      <xacro:property name="mat" value="0.25 0.25 0.25 1.0" />
     </xacro:if>
     <xacro:if value="${model == 'zedx'}">
@@ -69,4 +72,15 @@
       <xacro:property name="optical_offset_x" value="-0.01" />
       <xacro:property name="mono" value="false" />
+      <xacro:property name="mat" value="0.25 0.25 0.25 1.0" />
+    </xacro:if>
+    <xacro:if value="${model == 'zedxhdr'}">
+      <xacro:property name="baseline" value="0.12" />
+      <xacro:property name="height" value="0.032" />
+      <xacro:property name="bottom_slope" value="0.0" />
+      <xacro:property name="screw_offset_x" value="0.0" />
+      <xacro:property name="screw_offset_z" value="-0.016" />
+      <xacro:property name="optical_offset_x" value="-0.01" />
+      <xacro:property name="mono" value="false" />
+      <xacro:property name="mat" value="0.25 0.25 0.25 1.0" />
     </xacro:if>
     <xacro:if value="${model == 'zedxm'}">
@@ -78,4 +92,25 @@
       <xacro:property name="optical_offset_x" value="-0.01" />
       <xacro:property name="mono" value="false" />
+      <xacro:property name="mat" value="0.25 0.25 0.25 1.0" />
+    </xacro:if>
+    <xacro:if value="${model == 'zedxhdrmini'}">
+      <xacro:property name="baseline" value="0.05" />
+      <xacro:property name="height" value="0.032" />
+      <xacro:property name="bottom_slope" value="0.0" />
+      <xacro:property name="screw_offset_x" value="0.0" />
+      <xacro:property name="screw_offset_z" value="-0.016" />
+      <xacro:property name="optical_offset_x" value="-0.01" />
+      <xacro:property name="mono" value="false" />
+      <xacro:property name="mat" value="0.25 0.25 0.25 1.0" />
+    </xacro:if>
+    <xacro:if value="${model == 'zedxhdrmax'}">
+      <xacro:property name="baseline" value="0.170" />
+      <xacro:property name="height" value="0.032" />
+      <xacro:property name="bottom_slope" value="0.0" />
+      <xacro:property name="screw_offset_x" value="0.0" />
+      <xacro:property name="screw_offset_z" value="-0.016" />
+      <xacro:property name="optical_offset_x" value="-0.01" />
+      <xacro:property name="mono" value="false" />
+      <xacro:property name="mat" value="0.25 0.25 0.25 1.0" />
     </xacro:if>
     <xacro:if value="${model == 'virtual'}">
@@ -87,4 +122,5 @@
       <xacro:property name="optical_offset_x" value="0.0" />
       <xacro:property name="mono" value="false" />
+      <xacro:property name="mat" value="0.25 0.25 0.25 1.0" />
     </xacro:if>
     <xacro:if value="${model == 'zedxonegs'}">
@@ -96,4 +132,5 @@
       <xacro:property name="optical_offset_x" value="0.0" />
       <xacro:property name="mono" value="true" />
+      <xacro:property name="mat" value="0.25 0.25 0.25 1.0" />
     </xacro:if>
     <xacro:if value="${model == 'zedxone4k'}">
@@ -105,4 +142,15 @@
       <xacro:property name="optical_offset_x" value="0.0" />
       <xacro:property name="mono" value="true" />
+      <xacro:property name="mat" value="0.25 0.25 0.25 1.0" />
+    </xacro:if>
+    <xacro:if value="${model == 'zedxonehdr'}">
+      <xacro:property name="baseline" value="0.0" />
+      <xacro:property name="height" value="0.025" />
+      <xacro:property name="bottom_slope" value="0.0" />
+      <xacro:property name="screw_offset_x" value="0.00" />
+      <xacro:property name="screw_offset_z" value="-0.0125" />
+      <xacro:property name="optical_offset_x" value="0.0" />
+      <xacro:property name="mono" value="true" />
+      <xacro:property name="mat" value="0.25 0.25 0.25 1.0" />
     </xacro:if>
     <!-- Camera mounting point (the threaded screw hole in the bottom) -->
@@ -114,12 +162,14 @@
           <origin xyz="${screw_offset_x} 0 ${screw_offset_z}" rpy="0 0 0"/>
           <geometry>
-<mesh filename="file://$(find zed_msgs)/meshes/${model}.stl"/>
+            <mesh filename="file://$(find zed_msgs)/meshes/${model}.stl"/>
           </geometry>
-          <material name="${model}_mat" />
+            <material name="zed_mat">
+              <color rgba="${mat}"/>
+            </material>
         </visual>
         <collision>
           <origin xyz="${screw_offset_x} 0 ${screw_offset_z}" rpy="0 0 0"/>
           <geometry>
-<mesh filename="file://$(find zed_msgs)/meshes/${model}.stl"/>
+            <mesh filename="file://$(find zed_msgs)/meshes/${model}.stl"/>
           </geometry>
         </collision>
@@ -138,12 +188,14 @@
             <origin xyz="0 0 0" rpy="0 0 0"/>
             <geometry>
-  <mesh filename="file://$(find zed_msgs)/meshes/${model}.stl"/>
-            </geometry>
-            <material name="${model}_mat" />
+              <mesh filename="file://$(find zed_msgs)/meshes/${model}.stl"/>
+            </geometry>
+            <material name="zed_mat">
+              <color rgba="${mat}"/>
+            </material>
           </visual>
           <collision>
             <origin xyz="0 0 0" rpy="0 0 0"/>
             <geometry>
-  <mesh filename="file://$(find zed_msgs)/meshes/${model}.stl"/>
+              <mesh filename="file://$(find zed_msgs)/meshes/${model}.stl"/>
             </geometry>
           </collision>
@@ -155,9 +207,9 @@
         <origin xyz="${optical_offset_x} ${baseline/2} 0" rpy="0 0 0" />
       </joint>
-      <link name="${name}_left_camera_optical_frame"/>
+      <link name="${name}_left_camera_frame_optical"/>
       <joint name="${name}_left_camera_optical_joint" type="fixed">
         <origin xyz="0 0 0" rpy="-${M_PI/2} 0.0 -${M_PI/2}"/>
         <parent link="${name}_left_camera_frame"/>
-        <child link="${name}_left_camera_optical_frame"/>
+        <child link="${name}_left_camera_frame_optical"/>
       </joint>
       <!-- Right Camera -->
@@ -167,12 +219,14 @@
             <origin xyz="0 0 0" rpy="0 0 0"/>
             <geometry>
-  <mesh filename="file://$(find zed_msgs)/meshes/${model}.stl"/>
-            </geometry>
-            <material name="${model}_mat" />
+              <mesh filename="file://$(find zed_msgs)/meshes/${model}.stl"/>
+            </geometry>
+            <material name="zed_mat">
+              <color rgba="${mat}"/>
+            </material>
           </visual>
           <collision>
             <origin xyz="0 0 0" rpy="0 0 0"/>
             <geometry>
-  <mesh filename="file://$(find zed_msgs)/meshes/${model}.stl"/>
+              <mesh filename="file://$(find zed_msgs)/meshes/${model}.stl"/>
             </geometry>
           </collision>
@@ -184,9 +238,9 @@
         <origin xyz="${optical_offset_x} -${baseline/2} 0" rpy="0 0 0" />
       </joint>
-      <link name="${name}_right_camera_optical_frame"/>
+      <link name="${name}_right_camera_frame_optical"/>
       <joint name="${name}_right_camera_optical_joint" type="fixed">
         <origin xyz="0 0 0" rpy="-${M_PI/2} 0.0 -${M_PI/2}"/>
         <parent link="${name}_right_camera_frame"/>
-        <child link="${name}_right_camera_optical_frame"/>
+        <child link="${name}_right_camera_frame_optical"/>
       </joint>
       <!-- ZED2 Sensors -->
@@ -226,9 +280,9 @@
         <origin xyz="${optical_offset_x} 0 0" rpy="0 0 0" />
       </joint>
-      <link name="${name}_camera_optical_frame"/>
+      <link name="${name}_camera_frame_optical"/>
       <joint name="${name}_camera_optical_joint" type="fixed">
         <origin xyz="0 0 0" rpy="-${M_PI/2} 0.0 -${M_PI/2}"/>
         <parent link="${name}_camera_frame"/>
-        <child link="${name}_camera_optical_frame"/>
+        <child link="${name}_camera_frame_optical"/>
       </joint>
     </xacro:if>
