Commit message: feat: changes to fix the urdf to 6wd and also the new addresses and serial port

File: src/capybara_description/urdf/capybara.urdf.xacro (robot description, xacro)
@@ -1,4 +1,4 @@
 <?xml version="1.0"?>
-<robot name="gerbil" xmlns:xacro="http://www.ros.org/wiki/xacro">
+<robot name="capybara" xmlns:xacro="http://www.ros.org/wiki/xacro">
     <xacro:include filename="common_properties.xacro" />
     <xacro:include filename="mobile_base.xacro" />

File: src/capybara_description/urdf/mobile_base.ros2_control.xacro (robot description, xacro)
@@ -3,5 +3,5 @@
     <!-- Hardware mode - mock for simulation, real for actual RoboClaw -->
     <xacro:arg name="use_mock_hardware" default="true" />
-    <ros2_control name="GerbilRoboClawSystem" type="system">
+    <ros2_control name="CapybaraRoboClawSystem" type="system">
         <!-- Mock hardware for simulation or testing without actual RoboClaw -->
         <xacro:if value="$(arg use_mock_hardware)">
@@ -13,13 +13,12 @@
         <xacro:unless value="$(arg use_mock_hardware)">
             <hardware>
-                <plugin>gerbil_hw/RoboClawHardwareInterface</plugin>
-                <param name="serial_port">/dev/ttyTHS1</param>
+                <plugin>capybara_hw/RoboClawHardwareInterface</plugin>
+                <param name="serial_port">/dev/ttyTHS2</param>
                 <!-- Duty cycle mode - bypasses velocity PID, no encoders needed -->
-                <!-- Set to false once encoders are wired up -->
                 <param name="use_duty_cycle">true</param>
             </hardware>
         </xacro:unless>
-        <!-- joints that are defined and do not change whether using mock hardware or actual roboclaw hardware -->
-        <joint name="base_left_wheel_joint">
+        <!-- ==================== RoboClaw 128 (top): rear_right M1, front_left M2 ==================== -->
+        <joint name="front_left_wheel_joint">
             <command_interface name="velocity">
                 <param name="min">-10.0</param>
@@ -30,8 +29,7 @@
             <param name="qppr">500</param>
             <param name="motor_type">M2</param>
-            <!-- Motor speed (rad/s) that maps to 100 percent duty cycle. Lower = more responsive -->
             <param name="max_duty_speed">10.0</param>
         </joint>
-        <joint name="base_right_wheel_joint">
+        <joint name="rear_right_wheel_joint">
             <command_interface name="velocity">
                 <param name="min">-10.0</param>
@@ -42,5 +40,50 @@
             <param name="qppr">500</param>
             <param name="motor_type">M1</param>
-            <!-- Motor speed (rad/s) that maps to 100 percent duty cycle. Lower = more responsive -->
+            <param name="max_duty_speed">10.0</param>
+        </joint>
+        <!-- ==================== RoboClaw 129 (middle): mid_right M1, mid_left M2 ==================== -->
+        <joint name="mid_left_wheel_joint">
+            <command_interface name="velocity">
+                <param name="min">-10.0</param>
+                <param name="max">10.0</param>
+            </command_interface>
+            <state_interface name="position"/>
+            <param name="address">129</param>
+            <param name="qppr">500</param>
+            <param name="motor_type">M2</param>
+            <param name="max_duty_speed">10.0</param>
+        </joint>
+        <joint name="mid_right_wheel_joint">
+            <command_interface name="velocity">
+                <param name="min">-10.0</param>
+                <param name="max">10.0</param>
+            </command_interface>
+            <state_interface name="position"/>
+            <param name="address">129</param>
+            <param name="qppr">500</param>
+            <param name="motor_type">M1</param>
+            <param name="max_duty_speed">10.0</param>
+        </joint>
+        <!-- ==================== RoboClaw 130 (bottom): front_right M1, rear_left M2 ==================== -->
+        <joint name="rear_left_wheel_joint">
+            <command_interface name="velocity">
+                <param name="min">-10.0</param>
+                <param name="max">10.0</param>
+            </command_interface>
+            <state_interface name="position"/>
+            <param name="address">130</param>
+            <param name="qppr">500</param>
+            <param name="motor_type">M2</param>
+            <param name="max_duty_speed">10.0</param>
+        </joint>
+        <joint name="front_right_wheel_joint">
+            <command_interface name="velocity">
+                <param name="min">-10.0</param>
+                <param name="max">10.0</param>
+            </command_interface>
+            <state_interface name="position"/>
+            <param name="address">130</param>
+            <param name="qppr">500</param>
+            <param name="motor_type">M1</param>
             <param name="max_duty_speed">10.0</param>
         </joint>

File: src/capybara_description/urdf/mobile_base.xacro (robot description, xacro)
@@ -2,16 +2,28 @@
 <robot xmlns:xacro="http://www.ros.org/wiki/xacro">
     <!-- ROBOT DIMENSIONS -->
-    <!-- Drive wheels and ZED camera are at the front (+X) -->
-    <!-- Caster wheel is at the rear (-X) -->
-    <xacro:property name="base_length" value="0.6096" />      <!-- 24 inches -->
-    <xacro:property name="base_width" value="0.3048" />       <!-- 12 inches -->
-    <xacro:property name="base_height" value="0.0635" />      <!-- 2.5 inches -->
-    <xacro:property name="base_mass" value="6.8" />           <!-- ~15 lbs -->
-    <xacro:property name="wheel_radius" value="0.04756" />    <!-- 95.11mm diameter -->
-    <xacro:property name="wheel_length" value="0.03195" />    <!-- 31.95mm width -->
-    <xacro:property name="wheel_mass" value="0.5" />          <!-- kg estimate -->
-    <xacro:property name="wheel_separation" value="0.42285" /> <!-- 422.85mm center-to-center -->
-    <!-- Wheel X position - near front edge of chassis -->
-    <xacro:property name="wheel_x_offset" value="${base_length / 2.0 - 0.06}" />
+    <!-- TODO measure and update these values for the 6WD chassis -->
+    <xacro:property name="base_length" value="0.6096" />      <!-- 24 inches - UPDATE -->
+    <xacro:property name="base_width" value="0.3048" />       <!-- 12 inches - UPDATE -->
+    <xacro:property name="base_height" value="0.0635" />      <!-- 2.5 inches - UPDATE -->
+    <xacro:property name="base_mass" value="6.8" />           <!-- ~15 lbs - UPDATE -->
+    <!-- TODO measure wheel dimensions for 6WD chassis -->
+    <xacro:property name="wheel_radius" value="0.04756" />    <!-- UPDATE after measuring -->
+    <xacro:property name="wheel_length" value="0.03195" />    <!-- UPDATE after measuring -->
+    <xacro:property name="wheel_mass" value="0.5" />
+    <!-- Track widths - front/mid share one width, rear is wider -->
+    <!-- TODO measure both track widths -->
+    <xacro:property name="wheel_separation" value="0.42285" />       <!-- front+mid track width -->
+    <xacro:property name="rear_wheel_separation" value="0.48" />     <!-- rear track width - UPDATE -->
+    <!-- Axle X positions relative to base_link center -->
+    <!-- TODO measure axle spacing for 6WD chassis -->
+    <xacro:property name="front_axle_x" value="${base_length / 2.0 - 0.06}" />
+    <xacro:property name="mid_axle_x" value="0.0" />
+    <xacro:property name="rear_axle_x" value="${-base_length / 2.0 + 0.06}" />
+    <!-- LIDAR pole height (from chassis top to LIDAR center) -->
+    <!-- TODO measure the actual pole height -->
+    <xacro:property name="lidar_pole_height" value="0.25" />
+    <!-- Antenna stick height (from chassis top) -->
+    <xacro:property name="antenna_height" value="0.40" />
+    <xacro:property name="antenna_spacing" value="0.10" />
     <!-- BASE FOOTPRINT -->
     <link name="base_footprint" />
@@ -68,28 +80,12 @@
         </link>
     </xacro:macro>
-    <xacro:wheel_link prefix="right" />
-    <xacro:wheel_link prefix="left" />
-    <!-- CASTER WHEEL -->
-    <link name="caster_wheel_link">
-        <visual>
-            <geometry>
-                <sphere radius="${wheel_radius / 2.0}" />
-            </geometry>
-            <origin xyz="0 0 0" rpy="0 0 0" />
-            <material name="grey" />
-        </visual>
-        <collision>
-            <geometry>
-                <sphere radius="${wheel_radius / 2.0}" />
-            </geometry>
-            <origin xyz="0 0 0" rpy="0 0 0" />
-        </collision>
-        <inertial>
-            <mass value="0.2" />
-            <origin xyz="0 0 0" rpy="0 0 0" />
-            <inertia ixx="0.0001" ixy="0" ixz="0" iyy="0.0001" iyz="0" izz="0.0001" />
-        </inertial>
-    </link>
-    <!-- IMU LINK -->
+    <!-- 6 WHEELS -->
+    <xacro:wheel_link prefix="front_left" />
+    <xacro:wheel_link prefix="front_right" />
+    <xacro:wheel_link prefix="mid_left" />
+    <xacro:wheel_link prefix="mid_right" />
+    <xacro:wheel_link prefix="rear_left" />
+    <xacro:wheel_link prefix="rear_right" />
+    <!-- IMU LINK (ZED2i internal IMU) -->
     <link name="imu_link">
         <visual>
@@ -113,6 +109,4 @@
     </link>
     <!-- ZED2i CAMERA LINK -->
-    <!-- Named 'zed_camera_link' to match the ZED wrapper's TF frame,
-         connecting the robot URDF tree to the ZED's internal frame chain -->
     <link name="zed_camera_link">
         <visual>
@@ -135,5 +129,69 @@
         </inertial>
     </link>
-    <!-- JOINTS -->
+    <!-- LIDAR POLE (visual only, for collision awareness) -->
+    <link name="lidar_pole_link">
+        <visual>
+            <geometry>
+                <cylinder radius="0.01" length="${lidar_pole_height}" />
+            </geometry>
+            <origin xyz="0 0 0" rpy="0 0 0" />
+            <material name="grey" />
+        </visual>
+        <collision>
+            <geometry>
+                <cylinder radius="0.01" length="${lidar_pole_height}" />
+            </geometry>
+        </collision>
+        <inertial>
+            <mass value="0.1" />
+            <inertia ixx="0.000001" ixy="0" ixz="0" iyy="0.000001" iyz="0" izz="0.000001" />
+        </inertial>
+    </link>
+    <!-- LIDAR LINK (STL-19P) - on top of the pole -->
+    <link name="laser_frame">
+        <visual>
+            <geometry>
+                <cylinder radius="0.035" length="0.045" />
+            </geometry>
+            <origin xyz="0 0 0" rpy="0 0 0" />
+            <material name="dark_grey">
+                <color rgba="0.2 0.2 0.2 1" />
+            </material>
+        </visual>
+        <collision>
+            <geometry>
+                <cylinder radius="0.035" length="0.045" />
+            </geometry>
+        </collision>
+        <inertial>
+            <mass value="0.1" />
+            <inertia ixx="0.000001" ixy="0" ixz="0" iyy="0.000001" iyz="0" izz="0.000001" />
+        </inertial>
+    </link>
+    <!-- ANTENNA STICKS (rear of chassis, visual/collision only) -->
+    <xacro:macro name="antenna_link" params="prefix">
+        <link name="${prefix}_antenna_link">
+            <visual>
+                <geometry>
+                    <cylinder radius="0.005" length="${antenna_height}" />
+                </geometry>
+                <origin xyz="0 0 0" rpy="0 0 0" />
+                <material name="grey" />
+            </visual>
+            <collision>
+                <geometry>
+                    <cylinder radius="0.005" length="${antenna_height}" />
+                </geometry>
+            </collision>
+            <inertial>
+                <mass value="0.05" />
+                <inertia ixx="0.000001" ixy="0" ixz="0" iyy="0.000001" iyz="0" izz="0.000001" />
+            </inertial>
+        </link>
+    </xacro:macro>
+    <xacro:antenna_link prefix="left" />
+    <xacro:antenna_link prefix="right" />
+    <!-- ==================== JOINTS ==================== -->
+    <!-- Base footprint to base link -->
     <joint name="base_joint" type="fixed">
         <parent link="base_footprint" />
@@ -141,24 +199,23 @@
         <origin xyz="0 0 ${wheel_radius}" rpy="0 0 0"/>
     </joint>
-    <!-- Drive wheels at rear but changed to front -->
-    <joint name="base_right_wheel_joint" type="continuous">
-        <parent link="base_link" />
-        <child link="right_wheel_link" />
-        <origin xyz="${wheel_x_offset} ${-wheel_separation / 2.0} 0" rpy="0 0 0" />
-        <axis xyz="0 1 0" />
-    </joint>
-    <joint name="base_left_wheel_joint" type="continuous">
-        <parent link="base_link" />
-        <child link="left_wheel_link" />
-        <origin xyz="${wheel_x_offset} ${wheel_separation / 2.0} 0" rpy="0 0 0" />
-        <axis xyz="0 1 0" />
-    </joint>
-    <!-- Caster at the front, but we consider it rear -->
-    <joint name="base_caster_wheel_joint" type="fixed">
-        <parent link="base_link" />
-        <child link="caster_wheel_link" />
-        <origin xyz="${-wheel_x_offset} 0 ${-wheel_radius / 2.0}" rpy="0 0 0" />
-    </joint>
-    <!-- IMU centered on top of chassis not quite right, doesn't really matter, can add meshes later -->
+    <!-- WHEEL JOINT MACRO (takes per-axle separation) -->
+    <xacro:macro name="wheel_joint" params="prefix x_pos y_offset">
+        <joint name="${prefix}_wheel_joint" type="continuous">
+            <parent link="base_link" />
+            <child link="${prefix}_wheel_link" />
+            <origin xyz="${x_pos} ${y_offset} 0" rpy="0 0 0" />
+            <axis xyz="0 1 0" />
+        </joint>
+    </xacro:macro>
+    <!-- Front axle (standard width) -->
+    <xacro:wheel_joint prefix="front_left" x_pos="${front_axle_x}" y_offset="${wheel_separation / 2.0}" />
+    <xacro:wheel_joint prefix="front_right" x_pos="${front_axle_x}" y_offset="${-wheel_separation / 2.0}" />
+    <!-- Middle axle (standard width) -->
+    <xacro:wheel_joint prefix="mid_left" x_pos="${mid_axle_x}" y_offset="${wheel_separation / 2.0}" />
+    <xacro:wheel_joint prefix="mid_right" x_pos="${mid_axle_x}" y_offset="${-wheel_separation / 2.0}" />
+    <!-- Rear axle (wider) -->
+    <xacro:wheel_joint prefix="rear_left" x_pos="${rear_axle_x}" y_offset="${rear_wheel_separation / 2.0}" />
+    <xacro:wheel_joint prefix="rear_right" x_pos="${rear_axle_x}" y_offset="${-rear_wheel_separation / 2.0}" />
+    <!-- IMU centered on top of chassis -->
     <joint name="imu_joint" type="fixed">
         <parent link="base_link" />
@@ -166,5 +223,5 @@
         <origin xyz="0 0 ${base_height + 0.005}" rpy="0 0 0" />
     </joint>
-    <!-- ZED camera at front edge, on top of chassis, facing forward (rear) -->
+    <!-- ZED camera at front edge, on top of chassis, facing forward -->
     <joint name="camera_joint" type="fixed">
         <parent link="base_link" />
@@ -172,3 +229,26 @@
         <origin xyz="${base_length / 2.0 - 0.02} 0 ${base_height + 0.015}" rpy="0 0 0" />
     </joint>
+    <!-- LIDAR pole mounted center of chassis -->
+    <joint name="lidar_pole_joint" type="fixed">
+        <parent link="base_link" />
+        <child link="lidar_pole_link" />
+        <origin xyz="0 0 ${base_height + lidar_pole_height / 2.0}" rpy="0 0 0" />
+    </joint>
+    <!-- LIDAR on top of pole -->
+    <joint name="lidar_joint" type="fixed">
+        <parent link="base_link" />
+        <child link="laser_frame" />
+        <origin xyz="0 0 ${base_height + lidar_pole_height + 0.023}" rpy="0 0 0" />
+    </joint>
+    <!-- Antenna sticks at rear of chassis -->
+    <joint name="left_antenna_joint" type="fixed">
+        <parent link="base_link" />
+        <child link="left_antenna_link" />
+        <origin xyz="${rear_axle_x} ${antenna_spacing / 2.0} ${base_height + antenna_height / 2.0}" rpy="0 0 0" />
+    </joint>
+    <joint name="right_antenna_joint" type="fixed">
+        <parent link="base_link" />
+        <child link="right_antenna_link" />
+        <origin xyz="${rear_axle_x} ${-antenna_spacing / 2.0} ${base_height + antenna_height / 2.0}" rpy="0 0 0" />
+    </joint>
 </robot>

Commit message: changes to urdf to fix new layout of zed2i urdf based on new sdk

File: src/capybara_description/urdf/capybara.urdf.xacro (robot description, xacro)
@@ -4,3 +4,10 @@
     <xacro:include filename="mobile_base.xacro" />
     <xacro:include filename="mobile_base.ros2_control.xacro" />
+    <!-- ZED2i camera: provides zed_camera_link + all optical frame static TF.
+         publish_urdf:=false in capybara.launch.xml keeps the ZED RSP off so this
+         single capybara RSP is the sole owner of all static transforms. -->
+    <xacro:include filename="$(find zed_wrapper)/urdf/zed_macro.urdf.xacro" />
+    <xacro:zed_camera name="zed" model="zed2i">
+        <origin xyz="0 0 0" rpy="0 0 0"/>
+    </xacro:zed_camera>
 </robot>

File: src/capybara_description/urdf/mobile_base.xacro (robot description, xacro)
@@ -18,5 +18,5 @@
     <xacro:property name="rear_axle_x"  value="-0.4572" />    <!-- -18 inches from center -->
     <!-- LIDAR pole height from chassis top surface to LIDAR center -->
-    <xacro:property name="lidar_pole_height" value="0.508" />  <!-- 20 inches -->
+    <xacro:property name="lidar_pole_height" value="0.0254" />  <!-- 1 inch above chassis -->
     <!-- Antenna heights measured from chassis bottom (two different antennas) -->
     <xacro:property name="left_antenna_height"  value="0.762"  />  <!-- 2.4 GHz — 30 inches, left rear -->
@@ -104,25 +104,4 @@
         </inertial>
     </link>
-    <!-- ZED2i CAMERA LINK (named zed_camera_link to match ZED SDK v5 default camera_name='zed') -->
-    <link name="zed_camera_link">
-        <visual>
-            <geometry>
-                <box size="0.033 0.175 0.030" />
-            </geometry>
-            <origin xyz="0 0 0" rpy="0 0 0" />
-            <material name="dark_grey">
-                <color rgba="0.2 0.2 0.2 1" />
-            </material>
-        </visual>
-        <collision>
-            <geometry>
-                <box size="0.033 0.175 0.030" />
-            </geometry>
-        </collision>
-        <inertial>
-            <mass value="0.175" />
-            <inertia ixx="0.000001" ixy="0" ixz="0" iyy="0.000001" iyz="0" izz="0.000001" />
-        </inertial>
-    </link>
     <!-- LIDAR POLE (visual only, for collision awareness) -->
     <link name="lidar_pole_link">

Commit message: urdf changes to match lidar/gnss/ze2i change with lidar now

File: src/capybara_description/urdf/capybara.urdf.xacro (robot description, xacro)
@@ -4,6 +4,6 @@
     <xacro:include filename="mobile_base.xacro" />
     <xacro:include filename="mobile_base.ros2_control.xacro" />
-    <!-- ZED2i camera: provides zed_camera_link + all optical frame static TF.
-         publish_urdf:=false in capybara.launch.xml keeps the ZED RSP off so this
+    <!-- ZED2i camera — provides zed_camera_link and all optical frame static TF.
+         publish_urdf set to false in capybara.launch.xml keeps the ZED RSP off so this
          single capybara RSP is the sole owner of all static transforms. -->
     <xacro:include filename="$(find zed_wrapper)/urdf/zed_macro.urdf.xacro" />

File: src/capybara_description/urdf/mobile_base.xacro (robot description, xacro)
@@ -3,6 +3,6 @@
     <!-- ROBOT DIMENSIONS (measured Feb 2026, all values in meters) -->
     <xacro:property name="base_length" value="0.7112" />      <!-- 28 inches -->
-    <xacro:property name="base_width"  value="0.508"  />      <!-- 20 inches -->
-    <xacro:property name="base_height" value="0.1524" />      <!-- 6 inches  -->
+    <xacro:property name="base_width"  value="0.465"  />      <!-- 46.5 cm -->
+    <xacro:property name="base_height" value="0.26"   />      <!-- 26 cm     -->
     <xacro:property name="base_mass"   value="6.8"    />      <!-- ~15 lbs estimate -->
     <!-- Wheel dimensions (5 in radius including treads+rims, 3.5 in thick) -->
@@ -11,6 +11,6 @@
     <xacro:property name="wheel_mass"   value="0.5"    />
     <!-- Track widths center-of-left-wheel to center-of-right-wheel -->
-    <xacro:property name="wheel_separation"      value="0.762"  />  <!-- 30 in — front + mid axles -->
-    <xacro:property name="rear_wheel_separation" value="0.9144" />  <!-- 36 in — rear axle (wider) -->
+    <xacro:property name="wheel_separation"      value="0.6985" />  <!-- 27.5 in — all axles same -->
+    <xacro:property name="rear_wheel_separation" value="0.6985" />  <!-- 27.5 in — same as front/mid -->
     <!-- Axle X positions (mid axle = chassis center; 18 in = 0.4572 m between each adjacent pair) -->
     <xacro:property name="front_axle_x" value="0.4572"  />    <!-- +18 inches from center -->
@@ -18,5 +18,6 @@
     <xacro:property name="rear_axle_x"  value="-0.4572" />    <!-- -18 inches from center -->
     <!-- LIDAR pole height from chassis top surface to LIDAR center -->
-    <xacro:property name="lidar_pole_height" value="0.0254" />  <!-- 1 inch above chassis -->
+    <!-- Total lidar height from ground = 24in (0.6096m) = wheel_radius(0.127) + base_height(0.26) + pole + lidar_body_offset(0.023) -->
+    <xacro:property name="lidar_pole_height" value="0.1996" />  <!-- puts lidar at 24in from ground -->
     <!-- Antenna heights measured from chassis bottom (two different antennas) -->
     <xacro:property name="left_antenna_height"  value="0.762"  />  <!-- 2.4 GHz — 30 inches, left rear -->
@@ -200,12 +201,11 @@
     </joint>
     <!-- ZED SDK v5 zed_camera_link is the TF root (odom -> zed_camera_link published by ZED node).
-         base_footprint is now a child of zed_camera_link, at the inverse of the old mount offset.
-         Old mount base_link->(+0.3556, 0, +0.0762), base_joint->(0, 0, +0.127)
-         => camera was at (0.3556, 0, 0.2032) in base_footprint frame
-         => base_footprint is at (-0.3556, 0, -0.2032) in zed_camera_link frame -->
+         base_footprint is now a child of zed_camera_link, at the inverse of the camera mount offset.
+         Camera is 16.5in (0.4191m) forward of chassis center, 18.5in (0.4699m) above ground.
+         => base_footprint (ground level) is at (-0.4191, 0, -0.4699) in zed_camera_link frame -->
     <joint name="camera_footprint_joint" type="fixed">
         <parent link="zed_camera_link" />
         <child link="base_footprint" />
-        <origin xyz="-${base_length / 2.0} 0 -${wheel_radius + 0.0762}" rpy="0 0 0" />
+        <origin xyz="-0.4191 0 -0.4699" rpy="0 0 0" />
     </joint>
     <!-- LIDAR pole mounted center of chassis -->
