Commit message: update the urdf to be accurate, helps with open-loop movement apparently

File: src/capybara_description/urdf/mobile_base.xacro (robot description, xacro)
@@ -1,29 +1,25 @@
 <?xml version="1.0"?>
 <robot xmlns:xacro="http://www.ros.org/wiki/xacro">
-    <!-- ROBOT DIMENSIONS -->
-    <!-- TODO measure and update these values for the 6WD chassis -->
-    <xacro:property name="base_length" value="0.6096" />      <!-- 24 inches - UPDATE -->
-    <xacro:property name="base_width" value="0.3048" />       <!-- 12 inches - UPDATE -->
-    <xacro:property name="base_height" value="0.0635" />      <!-- 2.5 inches - UPDATE -->
-    <xacro:property name="base_mass" value="6.8" />           <!-- ~15 lbs - UPDATE -->
-    <!-- TODO measure wheel dimensions for 6WD chassis -->
-    <xacro:property name="wheel_radius" value="0.04756" />    <!-- UPDATE after measuring -->
-    <xacro:property name="wheel_length" value="0.03195" />    <!-- UPDATE after measuring -->
-    <xacro:property name="wheel_mass" value="0.5" />
-    <!-- Track widths - front/mid share one width, rear is wider -->
-    <!-- TODO measure both track widths -->
-    <xacro:property name="wheel_separation" value="0.42285" />       <!-- front+mid track width -->
-    <xacro:property name="rear_wheel_separation" value="0.48" />     <!-- rear track width - UPDATE -->
-    <!-- Axle X positions relative to base_link center -->
-    <!-- TODO measure axle spacing for 6WD chassis -->
-    <xacro:property name="front_axle_x" value="${base_length / 2.0 - 0.06}" />
-    <xacro:property name="mid_axle_x" value="0.0" />
-    <xacro:property name="rear_axle_x" value="${-base_length / 2.0 + 0.06}" />
-    <!-- LIDAR pole height (from chassis top to LIDAR center) -->
-    <!-- TODO measure the actual pole height -->
-    <xacro:property name="lidar_pole_height" value="0.25" />
-    <!-- Antenna stick height (from chassis top) -->
-    <xacro:property name="antenna_height" value="0.40" />
-    <xacro:property name="antenna_spacing" value="0.10" />
+    <!-- ROBOT DIMENSIONS (measured Feb 2026, all values in meters) -->
+    <xacro:property name="base_length" value="0.7112" />      <!-- 28 inches -->
+    <xacro:property name="base_width"  value="0.508"  />      <!-- 20 inches -->
+    <xacro:property name="base_height" value="0.1524" />      <!-- 6 inches  -->
+    <xacro:property name="base_mass"   value="6.8"    />      <!-- ~15 lbs estimate -->
+    <!-- Wheel dimensions (5 in radius including treads+rims, 3.5 in thick) -->
+    <xacro:property name="wheel_radius" value="0.127"  />     <!-- 5 inches  -->
+    <xacro:property name="wheel_length" value="0.0889" />     <!-- 3.5 inches -->
+    <xacro:property name="wheel_mass"   value="0.5"    />
+    <!-- Track widths: center-of-left-wheel to center-of-right-wheel -->
+    <xacro:property name="wheel_separation"      value="0.762"  />  <!-- 30 in — front + mid axles -->
+    <xacro:property name="rear_wheel_separation" value="0.9144" />  <!-- 36 in — rear axle (wider) -->
+    <!-- Axle X positions (mid axle = chassis center; 18 in = 0.4572 m between each pair) -->
+    <xacro:property name="front_axle_x" value="0.2286"  />    <!-- +9 inches from center -->
+    <xacro:property name="mid_axle_x"   value="0.0"     />
+    <xacro:property name="rear_axle_x"  value="-0.2286" />    <!-- -9 inches from center -->
+    <!-- LIDAR pole: height from chassis top surface to LIDAR center -->
+    <xacro:property name="lidar_pole_height" value="0.508" />  <!-- 20 inches -->
+    <!-- Antenna heights measured from chassis bottom (two different antennas) -->
+    <xacro:property name="left_antenna_height"  value="0.762"  />  <!-- 2.4 GHz — 30 inches, left rear -->
+    <xacro:property name="right_antenna_height" value="0.9144" />  <!-- 900 MHz  — 36 inches, right rear -->
     <!-- BASE FOOTPRINT -->
     <link name="base_footprint" />
@@ -170,9 +166,10 @@
     </link>
     <!-- ANTENNA STICKS (rear of chassis, visual/collision only) -->
-    <xacro:macro name="antenna_link" params="prefix">
+    <!-- Left = 2.4 GHz (30 in), Right = 900 MHz (36 in) — different heights -->
+    <xacro:macro name="antenna_link" params="prefix height">
         <link name="${prefix}_antenna_link">
             <visual>
                 <geometry>
-                    <cylinder radius="0.005" length="${antenna_height}" />
+                    <cylinder radius="0.005" length="${height}" />
                 </geometry>
                 <origin xyz="0 0 0" rpy="0 0 0" />
@@ -181,5 +178,5 @@
             <collision>
                 <geometry>
-                    <cylinder radius="0.005" length="${antenna_height}" />
+                    <cylinder radius="0.005" length="${height}" />
                 </geometry>
             </collision>
@@ -190,6 +187,6 @@
         </link>
     </xacro:macro>
-    <xacro:antenna_link prefix="left" />
-    <xacro:antenna_link prefix="right" />
+    <xacro:antenna_link prefix="left"  height="${left_antenna_height}"  />
+    <xacro:antenna_link prefix="right" height="${right_antenna_height}" />
     <!-- ==================== JOINTS ==================== -->
     <!-- Base footprint to base link -->
@@ -223,9 +220,9 @@
         <origin xyz="0 0 ${base_height + 0.005}" rpy="0 0 0" />
     </joint>
-    <!-- ZED camera at front edge, on top of chassis, facing forward -->
+    <!-- ZED2i: embedded in center of front panel, 3 in (0.0762 m) above chassis bottom -->
     <joint name="camera_joint" type="fixed">
         <parent link="base_link" />
         <child link="zed_camera_link" />
-        <origin xyz="${base_length / 2.0 - 0.02} 0 ${base_height + 0.015}" rpy="0 0 0" />
+        <origin xyz="${base_length / 2.0} 0 0.0762" rpy="0 0 0" />
     </joint>
     <!-- LIDAR pole mounted center of chassis -->
@@ -241,14 +238,15 @@
         <origin xyz="0 0 ${base_height + lidar_pole_height + 0.023}" rpy="0 0 0" />
     </joint>
-    <!-- Antenna sticks at rear of chassis -->
+    <!-- 2.4 GHz antenna: left side of back face, base at chassis bottom, rising upward -->
     <joint name="left_antenna_joint" type="fixed">
         <parent link="base_link" />
         <child link="left_antenna_link" />
-        <origin xyz="${rear_axle_x} ${antenna_spacing / 2.0} ${base_height + antenna_height / 2.0}" rpy="0 0 0" />
-    </joint>
+        <origin xyz="${-base_length / 2.0} ${base_width / 2.0} ${left_antenna_height / 2.0}" rpy="0 0 0" />
+    </joint>
+    <!-- 900 MHz antenna: right side of back face, base at chassis bottom, rising upward -->
     <joint name="right_antenna_joint" type="fixed">
         <parent link="base_link" />
         <child link="right_antenna_link" />
-        <origin xyz="${rear_axle_x} ${-antenna_spacing / 2.0} ${base_height + antenna_height / 2.0}" rpy="0 0 0" />
+        <origin xyz="${-base_length / 2.0} ${-base_width / 2.0} ${right_antenna_height / 2.0}" rpy="0 0 0" />
     </joint>
 </robot>

Commit message: feat: open-loop, fixed udrf for accurate dimensions

File: src/capybara_description/urdf/mobile_base.xacro (robot description, xacro)
@@ -10,12 +10,12 @@
     <xacro:property name="wheel_length" value="0.0889" />     <!-- 3.5 inches -->
     <xacro:property name="wheel_mass"   value="0.5"    />
-    <!-- Track widths: center-of-left-wheel to center-of-right-wheel -->
+    <!-- Track widths center-of-left-wheel to center-of-right-wheel -->
     <xacro:property name="wheel_separation"      value="0.762"  />  <!-- 30 in — front + mid axles -->
     <xacro:property name="rear_wheel_separation" value="0.9144" />  <!-- 36 in — rear axle (wider) -->
-    <!-- Axle X positions (mid axle = chassis center; 18 in = 0.4572 m between each pair) -->
-    <xacro:property name="front_axle_x" value="0.2286"  />    <!-- +9 inches from center -->
+    <!-- Axle X positions (mid axle = chassis center; 18 in = 0.4572 m between each adjacent pair) -->
+    <xacro:property name="front_axle_x" value="0.4572"  />    <!-- +18 inches from center -->
     <xacro:property name="mid_axle_x"   value="0.0"     />
-    <xacro:property name="rear_axle_x"  value="-0.2286" />    <!-- -9 inches from center -->
-    <!-- LIDAR pole: height from chassis top surface to LIDAR center -->
+    <xacro:property name="rear_axle_x"  value="-0.4572" />    <!-- -18 inches from center -->
+    <!-- LIDAR pole height from chassis top surface to LIDAR center -->
     <xacro:property name="lidar_pole_height" value="0.508" />  <!-- 20 inches -->
     <!-- Antenna heights measured from chassis bottom (two different antennas) -->
@@ -220,5 +220,5 @@
         <origin xyz="0 0 ${base_height + 0.005}" rpy="0 0 0" />
     </joint>
-    <!-- ZED2i: embedded in center of front panel, 3 in (0.0762 m) above chassis bottom -->
+    <!-- ZED2i embedded in center of front panel, 3 in (0.0762 m) above chassis bottom -->
     <joint name="camera_joint" type="fixed">
         <parent link="base_link" />
@@ -238,5 +238,5 @@
         <origin xyz="0 0 ${base_height + lidar_pole_height + 0.023}" rpy="0 0 0" />
     </joint>
-    <!-- 2.4 GHz antenna: left side of back face, base at chassis bottom, rising upward -->
+    <!-- 2.4 GHz antenna left side of back face, base at chassis bottom, rising upward -->
     <joint name="left_antenna_joint" type="fixed">
         <parent link="base_link" />
@@ -244,5 +244,5 @@
         <origin xyz="${-base_length / 2.0} ${base_width / 2.0} ${left_antenna_height / 2.0}" rpy="0 0 0" />
     </joint>
-    <!-- 900 MHz antenna: right side of back face, base at chassis bottom, rising upward -->
+    <!-- 900 MHz antenna right side of back face, base at chassis bottom, rising upward -->
     <joint name="right_antenna_joint" type="fixed">
         <parent link="base_link" />

Commit message: updated urdf errors caused by new urdf setup in SDK v5.2

File: src/capybara_description/urdf/mobile_base.xacro (robot description, xacro)
@@ -104,5 +104,5 @@
         </inertial>
     </link>
-    <!-- ZED2i CAMERA LINK -->
+    <!-- ZED2i CAMERA LINK (named zed_camera_link to match ZED SDK v5 default camera_name='zed') -->
     <link name="zed_camera_link">
         <visual>
@@ -220,9 +220,13 @@
         <origin xyz="0 0 ${base_height + 0.005}" rpy="0 0 0" />
     </joint>
-    <!-- ZED2i embedded in center of front panel, 3 in (0.0762 m) above chassis bottom -->
-    <joint name="camera_joint" type="fixed">
-        <parent link="base_link" />
-        <child link="zed_camera_link" />
-        <origin xyz="${base_length / 2.0} 0 0.0762" rpy="0 0 0" />
+    <!-- ZED SDK v5 zed_camera_link is the TF root (odom -> zed_camera_link published by ZED node).
+         base_footprint is now a child of zed_camera_link, at the inverse of the old mount offset.
+         Old mount base_link->(+0.3556, 0, +0.0762), base_joint->(0, 0, +0.127)
+         => camera was at (0.3556, 0, 0.2032) in base_footprint frame
+         => base_footprint is at (-0.3556, 0, -0.2032) in zed_camera_link frame -->
+    <joint name="camera_footprint_joint" type="fixed">
+        <parent link="zed_camera_link" />
+        <child link="base_footprint" />
+        <origin xyz="-${base_length / 2.0} 0 -${wheel_radius + 0.0762}" rpy="0 0 0" />
     </joint>
     <!-- LIDAR pole mounted center of chassis -->

Commit message: fix: removed imu link and made changes to lidar pole length to reflect actual rover

File: src/capybara_description/urdf/mobile_base.xacro (robot description, xacro)
@@ -17,6 +17,4 @@
     <xacro:property name="mid_axle_x"   value="0.0"     />
     <xacro:property name="rear_axle_x"  value="-0.4572" />    <!-- -18 inches from center -->
-    <!-- LIDAR pole height from chassis top surface to LIDAR center -->
-    <xacro:property name="lidar_pole_height" value="0.508" />  <!-- 20 inches -->
     <!-- Antenna heights measured from chassis bottom (two different antennas) -->
     <xacro:property name="left_antenna_height"  value="0.762"  />  <!-- 2.4 GHz — 30 inches, left rear -->
@@ -83,25 +81,4 @@
     <xacro:wheel_link prefix="rear_left" />
     <xacro:wheel_link prefix="rear_right" />
-    <!-- IMU LINK (ZED2i internal IMU) -->
-    <link name="imu_link">
-        <visual>
-            <geometry>
-                <box size="0.03 0.03 0.01" />
-            </geometry>
-            <origin xyz="0 0 0" rpy="0 0 0" />
-            <material name="green">
-                <color rgba="0 1 0 1" />
-            </material>
-        </visual>
-        <collision>
-            <geometry>
-                <box size="0.03 0.03 0.01" />
-            </geometry>
-        </collision>
-        <inertial>
-            <mass value="0.01" />
-            <inertia ixx="0.000001" ixy="0" ixz="0" iyy="0.000001" iyz="0" izz="0.000001" />
-        </inertial>
-    </link>
     <!-- ZED2i CAMERA LINK (named zed_camera_link to match ZED SDK v5 default camera_name='zed') -->
     <link name="zed_camera_link">
@@ -122,23 +99,4 @@
         <inertial>
             <mass value="0.175" />
-            <inertia ixx="0.000001" ixy="0" ixz="0" iyy="0.000001" iyz="0" izz="0.000001" />
-        </inertial>
-    </link>
-    <!-- LIDAR POLE (visual only, for collision awareness) -->
-    <link name="lidar_pole_link">
-        <visual>
-            <geometry>
-                <cylinder radius="0.01" length="${lidar_pole_height}" />
-            </geometry>
-            <origin xyz="0 0 0" rpy="0 0 0" />
-            <material name="grey" />
-        </visual>
-        <collision>
-            <geometry>
-                <cylinder radius="0.01" length="${lidar_pole_height}" />
-            </geometry>
-        </collision>
-        <inertial>
-            <mass value="0.1" />
             <inertia ixx="0.000001" ixy="0" ixz="0" iyy="0.000001" iyz="0" izz="0.000001" />
         </inertial>
@@ -214,10 +172,4 @@
     <xacro:wheel_joint prefix="rear_left" x_pos="${rear_axle_x}" y_offset="${rear_wheel_separation / 2.0}" />
     <xacro:wheel_joint prefix="rear_right" x_pos="${rear_axle_x}" y_offset="${-rear_wheel_separation / 2.0}" />
-    <!-- IMU centered on top of chassis -->
-    <joint name="imu_joint" type="fixed">
-        <parent link="base_link" />
-        <child link="imu_link" />
-        <origin xyz="0 0 ${base_height + 0.005}" rpy="0 0 0" />
-    </joint>
     <!-- ZED SDK v5 zed_camera_link is the TF root (odom -> zed_camera_link published by ZED node).
          base_footprint is now a child of zed_camera_link, at the inverse of the old mount offset.
@@ -230,15 +182,9 @@
         <origin xyz="-${base_length / 2.0} 0 -${wheel_radius + 0.0762}" rpy="0 0 0" />
     </joint>
-    <!-- LIDAR pole mounted center of chassis -->
-    <joint name="lidar_pole_joint" type="fixed">
-        <parent link="base_link" />
-        <child link="lidar_pole_link" />
-        <origin xyz="0 0 ${base_height + lidar_pole_height / 2.0}" rpy="0 0 0" />
-    </joint>
-    <!-- LIDAR on top of pole -->
+    <!-- LIDAR sitting directly on chassis top (no pole yet — placeholder until pole is fabricated) -->
     <joint name="lidar_joint" type="fixed">
         <parent link="base_link" />
         <child link="laser_frame" />
-        <origin xyz="0 0 ${base_height + lidar_pole_height + 0.023}" rpy="0 0 0" />
+        <origin xyz="0 0 ${base_height + 0.023}" rpy="0 0 0" />
     </joint>
     <!-- 2.4 GHz antenna left side of back face, base at chassis bottom, rising upward -->

Commit message: fix: changing lidar orientation in URDF and error message where SLAM cant find lidar scannings because of variable launch times

File: src/capybara_description/urdf/mobile_base.xacro (robot description, xacro)
@@ -186,5 +186,5 @@
         <parent link="base_link" />
         <child link="laser_frame" />
-        <origin xyz="0 0 ${base_height + 0.023}" rpy="0 0 0" />
+        <origin xyz="0 0 ${base_height + 0.023}" rpy="0 0 ${pi}" />
     </joint>
     <!-- 2.4 GHz antenna left side of back face, base at chassis bottom, rising upward -->

Commit message: test: fixing lidar urdf,orientation issues

File: src/capybara_description/urdf/mobile_base.xacro (robot description, xacro)
@@ -186,6 +186,5 @@
         <parent link="base_link" />
         <child link="laser_frame" />
-        <!-- 180 deg yaw because the sensor is mounted backwards relative to robot-forward. -->
-        <origin xyz="0 0 ${base_height + 0.023}" rpy="0 0 ${pi}" />
+        <origin xyz="0 0 ${base_height + 0.023}" rpy="0 0 0" />
     </joint>
     <!-- 2.4 GHz antenna left side of back face, base at chassis bottom, rising upward -->

Commit message: fix: shift lidar on urdf -1.5708 (90 degrees clockwise)

File: src/capybara_description/urdf/mobile_base.xacro (robot description, xacro)
@@ -186,5 +186,5 @@
         <parent link="base_link" />
         <child link="laser_frame" />
-        <origin xyz="0 0 ${base_height + 0.023}" rpy="0 0 0" />
+        <origin xyz="0 0 ${base_height + 0.023}" rpy="0 0 -1.5708" />
     </joint>
     <!-- 2.4 GHz antenna left side of back face, base at chassis bottom, rising upward -->
